File: macropad/pcb/macropad.kicad_sch (KiCad schematic)
At the start: 36 parts, among them J1 OLED_SSD1306, SW1 MX_Switch, SW10 MX_Switch, SW11 MX_Switch, SW12 MX_Switch, SW13 MX_Switch, SW14 MX_Switch, SW15 MX_Switch, SW16 MX_Switch, SW17 RESET, SW2 MX_Switch, SW3 MX_Switch, SW4 MX_Switch, SW5 MX_Switch, SW6 MX_Switch, SW7 MX_Switch, SW8 MX_Switch, SW9 MX_Switch, U1 Raspberry_Pi_Pico

Commit message: Fix schematic syntax errors for KiCad compatibility
Co-Authored-By: Claude Sonnet 4.6 <noreply@anthropic.com>
Parts:
- removed U1: Raspberry_Pi_Pico, MyCustLib:RPi_Pico_SMD, symbol MCU_RaspberryPi:RPi_Pico

Commit message: Simplify schematic to valid empty KiCad file
Co-Authored-By: Claude Sonnet 4.6 <noreply@anthropic.com>
Parts:
- removed D1, D10, D11, D12, D13, D14, D15, D16, D2, D3, D4, D5, D6, D7, D8, D9: 1N4148, Diode_THT:D_DO-35_SOD27_P7.62mm_Horizontal, symbol Device:D
- removed ENC1: EC11, Rotary_Encoder:RotaryEncoder_Alps_EC11E-Switch_Vertical_H20mm, symbol Device:Rotary_Encoder_Switch
- removed J1: OLED_SSD1306, Connector_PinHeader_2.54mm:PinHeader_1x04_P2.54mm_Vertical, symbol Connector:Conn_01x04_Pin
- removed SW1, SW10, SW11, SW12, SW13, SW14, SW15, SW16, SW2, SW3, SW4, SW5, SW6, SW7, SW8, SW9: MX_Switch, MX_Alps_Hybrid:MX-1U-NoLED, symbol Switch:SW_Push
- removed SW17: RESET, Button_Switch_THT:SW_SPST_PTS645, symbol Switch:SW_Push
